File: pcb/iron-hotplate.sch (EAGLE design)
At the start: 33 parts, among them CON1 KF301-2P, CON2 KF301-2P, Q1 AO3400, U1 EFM32GG11B420F2048GQ64, U2 MCP9601, U3 MIC23159, U4 LTV-354T-A

Commit message: Sync
Signed-off-by: João Silva <jgc3silva@gmail.com>
Parts:
- removed U3: MIC23159, Microchip:MIC23159
- added C107, C8, C88, C9: 100nF, Capacitor:CAPACITOR-0402
- added C108: 22uF, Capacitor:CAPACITOR-1206
- added C91: 4.7uF, Capacitor:CAPACITOR-0603
- added C97: 470pF, Capacitor:CAPACITOR-0402
- added D2, D3: BAV99, Generic Diode:BAV99
- added L1: 1.2uH, Coilcraft:XGL3512-122
- added R10: 487K Ohms, Resistor:RESISTOR-0402
- added R11, R12: 100 Ohms, Resistor:RESISTOR-0402
- added R49: 10K Ohms, Resistor:RESISTOR-0402
- added R52: 309K Ohms, Resistor:RESISTOR-0402
- added R53: 71.5K Ohms, Resistor:RESISTOR-0402
- added R8: 2M Ohms, Resistor:RESISTOR-0402
- added R9: 2.49M Ohms, Resistor:RESISTOR-0402
- added U18: MIC23155, Microchip:MIC23155
- U4: value LTV-354T-A -> K814P; device Generic Optocoupler:LTV-354T-A -> Generic Optocoupler:K814P
Connections:
- removed net 2V5: C110.C1, C2.C1, C3.C1, C4.C1, C5.C1, C6.C1
- new net 3V3_FB: R52.1, R53.2, U18.FB
- new net 3V3_PGOOD: R49.1, U18.PG
- new net 3V3_SS: C97.C1, U18.SS
- new net 3V3_SW: L1.1, U18.SW
- new net N$8: R11.2, U2.VIN+
- new net N$9: R12.2, U2.VIN-
- new net TC0_N: C8.C2, D2.MID, R10.2, R12.1
- new net TC0_P: C8.C1, D3.MID, R11.1, R8.1, R9.2, U2.VSENSE
- net 3V3: now also C107.C1, C108.C1, C110.C1, C2.C1, C3.C1, C4.C1, C5.C1, C6.C1, C9.C1, D2.C, D3.C, L1.2, R49.2, R52.2, R8.2, U18.SNS, U2.VDD
- net 5V0: now also C88.C1, C91.C1, U18.EN, U18.VIN@0, U18.VIN@1
- net GND: now also C107.C2, C108.C2, C88.C2, C9.C2, C91.C2, C97.C2, D2.A, D3.A, R10.1, R53.1, R9.1, U18.AGND, U18.PGND@0, U18.PGND@1, U2.GND
Other:
- moved on the sheet: U2
